Commit message: joint file coded up with undetermined values and small changes

File: src/moa/moa_description/moa_description/urdf/links.xacro (robot description, xacro)
@@ -5,5 +5,5 @@
     <link name='base_link'/>
     <!--chassis link-->
-    <link name='chassis'>
+    <link name='chassis_link'>
         <visual>
             <geometry>
@@ -15,21 +15,21 @@
     </link>
     <!--Wheel/Tyre link-->
-    <xacro:tyre_link name='front_right_wheel'>
+    <xacro:tyre_link name='front_right_wheel_link'>
         <origin xyz='A B C' rpy='A B C'/>
     </xacro:tyre_link>
-    <xacro:tyre_link name='front_left_wheel'>
+    <xacro:tyre_link name='front_left_wheel_link'>
         <origin xyz='A B C' rpy='A B C'/>
     </xacro:tyre_link>
-    <xacro:tyre_link name='rear_right_wheel'>
+    <xacro:tyre_link name='rear_right_wheel_link'>
         <origin xyz='A B C' rpy='A B C'/>
     </xacro:tyre_link>
-    <xacro:tyre_link name='rear_left_wheel'>
+    <xacro:tyre_link name='rear_left_wheel_link'>
         <origin xyz='A B C' rpy='A B C'/>
     </xacro:tyre_link>
     <!--kingpin link-->
-    <xacro:kingpin_link name='front_right_pin'>
+    <xacro:kingpin_link name='right_kingpin_link'>
         <origin xyz='A B C' rpy='A B C'/>
     </xacro:kingpin_link>
-    <xacro:kingpin_link name='front_left_pin'>
+    <xacro:kingpin_link name='left_kingpin_link'>
         <origin xyz='A B C' rpy='A B C'/>
     </xacro:kingpin_link>

File: src/moa/moa_description/moa_description/urdf/macro.xacro (robot description, xacro)
@@ -8,5 +8,5 @@
                 <xacro:insert_block name='origin'/>
                 <geometry>
-                    <mesh filename='package://moa_description/meshes/M023_Wheel.stl'/>
+                    <mesh filename='package://src/moa/moa_description/moa_description/meshes/M023_Wheel.stl'/>
                 </geometry>
             </visual>
