Commit message: small change - quick temp setup of values

File: src/moa/moa_description/moa_description/urdf/const.xacro (robot description, xacro)
@@ -3,3 +3,5 @@
 	<!--robot name-->
 	<xacro:property name='robot_name' value='moa23'/>
+	<!-- quick edit to set all origins/rpy-->
+	<xacro:property name='A B C' value='0 0 0'/>
 </robot>

File: src/moa/moa_description/moa_description/urdf/joints.xacro (robot description, xacro)
@@ -52,3 +52,3 @@
         <axis xyz='A B C'/>
     </joint>
-</robot>
+</robot>~
