Commit message: chassis mesh and zed docker image

File: src/moa/moa_description/urdf/links.xacro (robot description, xacro)
@@ -8,6 +8,6 @@
         <visual>
             <geometry>
-                <!--mesh filename='$ABC'-->
-                <box size='50 50 50'/>
+                <mesh filename='package://src/moa/moa_description/meshes/Body23.stl'/>
+                <!-- <box size='50 50 50'/> -->
             </geometry>
             <origin  xyz='0 0 0' rpy='0 0 0'/>

File: src/moa/moa_description/urdf/macro.xacro (robot description, xacro)
@@ -8,5 +8,5 @@
                 <xacro:insert_block name='origin'/>
                 <geometry>
-                    <mesh filename='package://src/moa/moa_description/meshes/M023_Wheel.stl'/>
+                    <mesh filename='package://moa_description/meshes/wheel.stl'/>
                 </geometry>
             </visual>

File: src/moa/moa_description/urdf/robot.urdf.xacro (robot description, xacro)
@@ -7,3 +7,5 @@
     <xacro:include filename="$(find moa_description)/urdf/links.xacro" />
     <xacro:include filename="$(find moa_description)/urdf/joints.xacro" />
+    <!-- camera urdf -->
+    <!-- <xacro:include filename='/ws/src/hardware_drivers/zed-ros2-wrapper/zed_wrapper/urdf/zed_descr.urdf.xacro'/> -->
 </robot>
