Commit message: moved some files

File: src/moa/moa_description/urdf/const.xacro (robot description, xacro)
@@ -4,4 +4,4 @@
 	<xacro:property name='robot_name' value='moa23'/>
 	<!-- quick edit to set all origins/rpy-->
-	<xacro:property name='A B C' value='0 0 0'/>
+	<!-- <xacro:property name='A B C' value='0 0 0'/> -->
 </robot>

File: src/moa/moa_description/urdf/joints.xacro (robot description, xacro)
@@ -7,5 +7,5 @@
         <child link='chassis_link'/>
         <!--the origin tag over here means the origin of the join before any motion/transformation occurs-->
-        <origin xyz='A B C' rpy='A B C'/>
+        <origin xyz='0 0 0' rpy='0 0 0'/>
     </joint>
     <!--Chassis to kingpin1 joint-->
@@ -13,7 +13,7 @@
         <parent link='chassis_link'/>
         <child link='right_kingpin_link'/>
-        <origin xyz='A B C' rpy='A B C'/>
-        <axis xyz='A B C'/>
-        <limit lower='-A' upper='+A' velocity='1' effot='25'/>
+        <origin xyz='0 0 0' rpy='0 0 0'/>
+        <axis xyz='0 0 0'/>
+        <limit lower='-0.44' upper='0.66' velocity='1' effot='25'/>
     </joint>
       <!--Chassis to kingpin2 joint-->
@@ -21,7 +21,7 @@
         <parent link='chassis_link'/>
         <child link='left_kingpin_link'/>
-        <origin xyz='A B C' rpy='A B C'/>
-        <axis xyz='A B C'/>
-        <limit lower='-A' upper='+A' velocity='1' effot='25'/>
+        <origin xyz='0 0 0' rpy='0 0 0'/>
+        <axis xyz='0 0 0'/>
+        <limit lower='-0.44' upper='0.66' velocity='1' effot='25'/>
     </joint>
     <!--Kingpin1 to wheel joint-->
@@ -30,5 +30,5 @@
         <child link='front_right_wheel_link'/>
         <!--steering wheel joints don't have origin as its at the kinpin link?-->
-        <axis xyz='A B C'/>
+        <axis xyz='0 1 0'/>
     </joint>
     <!--Kingpin2 to wheel joint-->
@@ -36,5 +36,5 @@
         <parent link='left_kingpin_link'/>
         <child link='front_left_wheel_link'/>
-        <axis xyz='A B C'/>
+        <axis xyz='0 1 0'/>
     </joint>
     <!--Chassis to wheel joint-->
@@ -42,6 +42,6 @@
         <parent link='chassis_link'/>
         <child link='rear_right_wheel_link'/>
-        <origin xyz='A B C' rpy='A B C'/>
-        <axis xyz='A B C'/>
+        <origin xyz='0 0 0' rpy='0 0 0'/>
+        <axis xyz='0 1 0'/>
     </joint>
     <!--Chassis to wheel joint-->
@@ -49,6 +49,6 @@
         <parent link='chassis_link'/>
         <child link='rear_left_wheel_link'/>
-        <origin xyz='A B C' rpy='A B C'/>
-        <axis xyz='A B C'/>
+        <origin xyz='0 0 0' rpy='0 0 0'/>
+        <axis xyz='0 1 0'/>
     </joint>
-</robot>~
+</robot>

File: src/moa/moa_description/urdf/links.xacro (robot description, xacro)
@@ -9,28 +9,28 @@
             <geometry>
                 <!--mesh filename='$ABC'-->
-                <box size='1000'/>
+                <box size='500'/>
             </geometry>
-            <origin  xyz='A B C' rpy='A B C'/>
+            <origin  xyz='0 0 0' rpy='0 0 0'/>
         </visual>
     </link>
     <!--Wheel/Tyre link-->
     <xacro:tyre_link name='front_right_wheel_link'>
-        <origin xyz='A B C' rpy='A B C'/>
+        <origin xyz='0 0 0' rpy='0 0 0'/>
     </xacro:tyre_link>
     <xacro:tyre_link name='front_left_wheel_link'>
-        <origin xyz='A B C' rpy='A B C'/>
+        <origin xyz='0 0 0' rpy='0 0 0'/>
     </xacro:tyre_link>
     <xacro:tyre_link name='rear_right_wheel_link'>
-        <origin xyz='A B C' rpy='A B C'/>
+        <origin xyz='0 0 0' rpy='0 0 0'/>
     </xacro:tyre_link>
     <xacro:tyre_link name='rear_left_wheel_link'>
-        <origin xyz='A B C' rpy='A B C'/>
+        <origin xyz='0 0 0' rpy='0 0 0'/>
     </xacro:tyre_link>
     <!--kingpin link-->
     <xacro:kingpin_link name='right_kingpin_link'>
-        <origin xyz='A B C' rpy='A B C'/>
+        <origin xyz='0 0 0' rpy='0 0 0'/>
     </xacro:kingpin_link>
     <xacro:kingpin_link name='left_kingpin_link'>
-        <origin xyz='A B C' rpy='A B C'/>
+        <origin xyz='0 0 0' rpy='0 0 0'/>
     </xacro:kingpin_link>
 </robot>

File: src/moa/moa_description/urdf/macro.xacro (robot description, xacro)
@@ -3,5 +3,5 @@
 <!--WHERE THERE IS 'ABC' IT MEANS THE VALUE OR FIELD IS NOT DETERMINED YET-->
     <!--wheel macro-->
-    <xacro:macro name="tyre_link" params="name, *origin">
+    <xacro:macro name="tyre_link" params="name *origin">
         <link name="${name}">
             <visual>

Commit message: value changes and config share folder for urdf files

File: src/moa/moa_description/urdf/const.xacro (robot description, xacro)
@@ -4,4 +4,3 @@
 	<xacro:property name='robot_name' value='moa23'/>
 	<!-- quick edit to set all origins/rpy-->
-	<!-- <xacro:property name='A B C' value='0 0 0'/> -->
 </robot>

File: src/moa/moa_description/urdf/joints.xacro (robot description, xacro)
@@ -15,5 +15,5 @@
         <origin xyz='0 0 0' rpy='0 0 0'/>
         <axis xyz='0 0 0'/>
-        <limit lower='-0.44' upper='0.66' velocity='1' effot='25'/>
+        <limit lower='-0.44' upper='0.66' velocity='1' effort='25'/>
     </joint>
       <!--Chassis to kingpin2 joint-->
@@ -23,5 +23,5 @@
         <origin xyz='0 0 0' rpy='0 0 0'/>
         <axis xyz='0 0 0'/>
-        <limit lower='-0.44' upper='0.66' velocity='1' effot='25'/>
+        <limit lower='-0.44' upper='0.66' velocity='1' effort='25'/>
     </joint>
     <!--Kingpin1 to wheel joint-->

File: src/moa/moa_description/urdf/links.xacro (robot description, xacro)
@@ -9,5 +9,5 @@
             <geometry>
                 <!--mesh filename='$ABC'-->
-                <box size='500'/>
+                <box size='50 50 50'/>
             </geometry>
             <origin  xyz='0 0 0' rpy='0 0 0'/>

File: src/moa/moa_description/urdf/macro.xacro (robot description, xacro)
@@ -8,5 +8,5 @@
                 <xacro:insert_block name='origin'/>
                 <geometry>
-                    <mesh filename='package://src/moa/moa_description/moa_description/meshes/M023_Wheel.stl'/>
+                    <mesh filename='package://src/moa/moa_description/meshes/M023_Wheel.stl'/>
                 </geometry>
             </visual>

Commit message: all coods to meteres with meters unit mesh files and material added

File: src/moa/moa_description/urdf/const.xacro (robot description, xacro)
@@ -3,4 +3,9 @@
 	<!--robot name-->
 	<xacro:property name='robot_name' value='moa23'/>
-	<!-- quick edit to set all origins/rpy-->
+	<!-- kingpin dimensions-->
+	<xacro:property name='kingpin_radius' value='0.003175'/>
+	<xacro:property name='kingpin_length' value='0.038213'/>
+	<!-- steering angles based on ackerman steering-->
+	<xacro:property name='steering_in' value='${25*pi/180}'/>
+	<xacro:property name='steering_out' value='${38*pi/180}'/>
 </robot>

File: src/moa/moa_description/urdf/joints.xacro (robot description, xacro)
@@ -1,11 +1,9 @@
 <?xml version="1.0"?>
 <robot xmlns:xacro="http://www.ros.org/wiki/xacro">
-<!--WHERE THERE IS 'ABC' IT MEANS THE VALUE OR FIELD IS NOT DETERMINED YET-->
     <!--base to chassis joint-->
     <joint name='base_to_chassis_joint' type='fixed'>
         <parent link='base_link'/>
         <child link='chassis_link'/>
-        <!--the origin tag over here means the origin of the join before any motion/transformation occurs-->
-        <origin xyz='0 0 0' rpy='0 0 0'/>
+        <origin xyz='-0.281 0 -0.133' rpy='0 0 0'/>
     </joint>
     <!--Chassis to kingpin1 joint-->
@@ -13,7 +11,7 @@
         <parent link='chassis_link'/>
         <child link='right_kingpin_link'/>
-        <origin xyz='0 0 0' rpy='0 0 0'/>
-        <axis xyz='0 0 0'/>
-        <limit lower='-0.44' upper='0.66' velocity='1' effort='25'/>
+        <origin xyz='0.288 0.571 -0.167' rpy='0 0 0'/>
+        <axis xyz='0 0 1'/>
+        <limit lower='${-steering_out}' upper='${steering_in}' velocity='1' effort='25'/>
     </joint>
       <!--Chassis to kingpin2 joint-->
@@ -21,7 +19,7 @@
         <parent link='chassis_link'/>
         <child link='left_kingpin_link'/>
-        <origin xyz='0 0 0' rpy='0 0 0'/>
-        <axis xyz='0 0 0'/>
-        <limit lower='-0.44' upper='0.66' velocity='1' effort='25'/>
+        <origin xyz='0.288 -0.571 -0.167' rpy='0 0 0'/>
+        <axis xyz='0 0 1'/>
+        <limit lower='${-steering_in}' upper='${steering_out}' velocity='1' effort='25'/>
     </joint>
     <!--Kingpin1 to wheel joint-->
@@ -29,5 +27,5 @@
         <parent link='right_kingpin_link'/>
         <child link='front_right_wheel_link'/>
-        <!--steering wheel joints don't have origin as its at the kinpin link?-->
+        <origin xyz='-0.007 0.065 0.087' rpy='0 0 0'/>
         <axis xyz='0 1 0'/>
     </joint>
@@ -36,4 +34,5 @@
         <parent link='left_kingpin_link'/>
         <child link='front_left_wheel_link'/>
+        <origin xyz='-0.007 -0.065 0.087' rpy='0 0 0'/>
         <axis xyz='0 1 0'/>
     </joint>
@@ -42,5 +41,5 @@
         <parent link='chassis_link'/>
         <child link='rear_right_wheel_link'/>
-        <origin xyz='0 0 0' rpy='0 0 0'/>
+        <origin xyz='-1.249 0.589 -0.077' rpy='0 0 0'/>
         <axis xyz='0 1 0'/>
     </joint>
@@ -49,5 +48,5 @@
         <parent link='chassis_link'/>
         <child link='rear_left_wheel_link'/>
-        <origin xyz='0 0 0' rpy='0 0 0'/>
+        <origin xyz='-1.249 -0.589 -0.077' rpy='0 0 0'/>
         <axis xyz='0 1 0'/>
     </joint>

File: src/moa/moa_description/urdf/links.xacro (robot description, xacro)
@@ -1,5 +1,4 @@
 <?xml version='1.0'?>
 <robot xmlns:xacro="http://www.ros.org/wiki/xacro">
-<!--WHERE THERE IS 'ABC' IT MEANS THE VALUE OR FIELD IS NOT DETERMINED YET-->
     <!--base link-->
     <link name='base_link'/>
@@ -8,22 +7,25 @@
         <visual>
             <geometry>
-                <mesh filename='package://src/moa/moa_description/meshes/Body23.stl'/>
-                <!-- <box size='50 50 50'/> -->
+                <mesh filename='package://moa_description/meshes/Chassis.stl'/>
             </geometry>
-            <origin  xyz='0 0 0' rpy='0 0 0'/>
+            <material name='grey'>
+                <color rgba='0.4 0.4 0.4 1'/>
+            </material>
+            <!--chassis link origin should be center of mass-->
+            <origin  xyz='0.281 0 0.133' rpy='${-pi/2} 0 0'/>
         </visual>
     </link>
     <!--Wheel/Tyre link-->
     <xacro:tyre_link name='front_right_wheel_link'>
-        <origin xyz='0 0 0' rpy='0 0 0'/>
+        <origin xyz='0 0 0' rpy='${pi/2} 0 0'/>
     </xacro:tyre_link>
     <xacro:tyre_link name='front_left_wheel_link'>
-        <origin xyz='0 0 0' rpy='0 0 0'/>
+        <origin xyz='0 0 0' rpy='${-pi/2} 0 0'/>
     </xacro:tyre_link>
     <xacro:tyre_link name='rear_right_wheel_link'>
-        <origin xyz='0 0 0' rpy='0 0 0'/>
+        <origin xyz='0 0 0' rpy='${pi/2} 0 0'/>
     </xacro:tyre_link>
     <xacro:tyre_link name='rear_left_wheel_link'>
-        <origin xyz='0 0 0' rpy='0 0 0'/>
+        <origin xyz='0 0 0' rpy='${-pi/2} 0 0'/>
     </xacro:tyre_link>
     <!--kingpin link-->

File: src/moa/moa_description/urdf/macro.xacro (robot description, xacro)
@@ -1,5 +1,4 @@
 <?xml version='1.0'?>
 <robot xmlns:xacro="http://www.ros.org/wiki/xacro">
-<!--WHERE THERE IS 'ABC' IT MEANS THE VALUE OR FIELD IS NOT DETERMINED YET-->
     <!--wheel macro-->
     <xacro:macro name="tyre_link" params="name *origin">
@@ -8,6 +7,9 @@
                 <xacro:insert_block name='origin'/>
                 <geometry>
-                    <mesh filename='package://moa_description/meshes/wheel.stl'/>
+                    <mesh filename='package://moa_description/meshes/Wheel.stl'/>
                 </geometry>
+                <material name='black'>
+                    <color rgba='0 0 0 1'/>
+                </material>
             </visual>
         </link>
@@ -19,5 +21,5 @@
                 <xacro:insert_block name='origin'/>
                 <geometry>
-                    <sphere radius='3'/>
+                    <cylinder radius='${kingpin_radius}' length='${kingpin_length}'/>
                 </geometry>
             </visual>
