Commit message: trying to setup gazebo and urdf

File: src/moa/moa_description/urdf/moa_macro.xacro (robot description, xacro)
@@ -7,5 +7,5 @@
                 <xacro:insert_block name='origin'/>
                 <geometry>
-                    <mesh filename='package://moa_description/meshes/Wheel.stl'/>
+                    <mesh filename='package://moa_description/meshes/wheel.stl'/>
                 </geometry>
                 <material name='black'>
@@ -13,4 +13,15 @@
                 </material>
             </visual>
+            <inertial>
+                <!-- <origin xyz="0.0 0.0 0.0" rpy="0.0 0.0 0.0"/> -->
+                <mass value="5.0"/>
+                <inertia ixx="0.0" ixy="0.0" ixz="0.0" iyy="0.0" iyz="0.0" izz="0.0"/>
+            </inertial>
+            <collision>
+                <xacro:insert_block name='origin'/>
+                <geometry>
+                    <mesh filename='package://moa_description/meshes/wheel.stl'/>
+                </geometry>
+            </collision>
         </link>
     </xacro:macro>

File: src/moa/moa_description/urdf/moa_robot.urdf.xacro (robot description, xacro)
@@ -9,3 +9,5 @@
     <xacro:include filename="$(find moa_description)/urdf/moa_links.xacro" />
     <xacro:include filename="$(find moa_description)/urdf/moa_joints.xacro" />
+    <!-- gazebo-->
+    <xacro:include filename='$(find moa_description)/urdf/gazebo.xacro' />
 </robot>
