Commit message: Zed camera urdf mounted properly - last commit potentially

File: src/moa/moa_description/urdf/moa_joints.xacro (robot description, xacro)
@@ -2,6 +2,6 @@
 <robot xmlns:xacro="http://www.ros.org/wiki/xacro">
     <!--base to chassis joint-->
-    <joint name='base_to_chassis_joint' type='fixed'>
-        <parent link='base_link'/>
+    <joint name='world_to_chassis_joint' type='fixed'>
+        <parent link='world_link'/>
         <child link='chassis_link'/>
         <origin xyz='-0.281 0 -0.133' rpy='0 0 0'/>
@@ -13,5 +13,5 @@
         <origin xyz='0.288 0.571 -0.167' rpy='0 0 0'/>
         <axis xyz='0 0 1'/>
-        <limit lower='${-steering_out}' upper='${steering_in}' velocity='1' effort='25'/>
+        <limit lower='${-steering_in}' upper='${steering_out}' velocity='1' effort='25'/>
     </joint>
       <!--Chassis to kingpin2 joint-->
@@ -21,5 +21,5 @@
         <origin xyz='0.288 -0.571 -0.167' rpy='0 0 0'/>
         <axis xyz='0 0 1'/>
-        <limit lower='${-steering_in}' upper='${steering_out}' velocity='1' effort='25'/>
+        <limit lower='${-steering_out}' upper='${steering_in}' velocity='1' effort='25'/>
     </joint>
     <!--Kingpin1 to wheel joint-->
@@ -51,3 +51,9 @@
         <axis xyz='0 1 0'/>
     </joint>
+    <!--world to zed base joint-->
+    <joint name='chassis_to_zed_base' type='fixed'>
+        <parent link='chassis_link'/>
+        <child link='base_link'/>
+        <origin xyz='-0.741 -0.002 -1.029' rpy='${-pi/2} 0 0'/>
+    </joint>
 </robot>

File: src/moa/moa_description/urdf/moa_links.xacro (robot description, xacro)
@@ -1,6 +1,6 @@
 <?xml version='1.0'?>
 <robot xmlns:xacro="http://www.ros.org/wiki/xacro">
-    <!--base link-->
-    <link name='base_link'/>
+    <!--world link-->
+    <link name='world_link'/>
     <!--chassis link-->
     <link name='chassis_link'>
@@ -12,5 +12,4 @@
                 <color rgba='0.4 0.4 0.4 1'/>
             </material>
-            <!--chassis link origin should be center of mass-->
             <origin  xyz='0.281 0 0.133' rpy='${-pi/2} 0 0'/>
         </visual>

Commit message: addressed review 1 and flipped z-axis for mesh

File: src/moa/moa_description/urdf/moa_joints.xacro (robot description, xacro)
@@ -5,5 +5,5 @@
         <parent link='world_link'/>
         <child link='chassis_link'/>
-        <origin xyz='-0.281 0 -0.133' rpy='0 0 0'/>
+        <origin xyz='-0.281 0 0.133' rpy='0 0 0'/>
     </joint>
     <!--Chassis to kingpin1 joint-->
@@ -11,5 +11,5 @@
         <parent link='chassis_link'/>
         <child link='right_kingpin_link'/>
-        <origin xyz='0.288 0.571 -0.167' rpy='0 0 0'/>
+        <origin xyz='0.288 0.571 0.167' rpy='0 0 0'/>
         <axis xyz='0 0 1'/>
         <limit lower='${-steering_in}' upper='${steering_out}' velocity='1' effort='25'/>
@@ -19,5 +19,5 @@
         <parent link='chassis_link'/>
         <child link='left_kingpin_link'/>
-        <origin xyz='0.288 -0.571 -0.167' rpy='0 0 0'/>
+        <origin xyz='0.288 -0.571 0.167' rpy='0 0 0'/>
         <axis xyz='0 0 1'/>
         <limit lower='${-steering_out}' upper='${steering_in}' velocity='1' effort='25'/>
@@ -27,5 +27,5 @@
         <parent link='right_kingpin_link'/>
         <child link='front_right_wheel_link'/>
-        <origin xyz='-0.007 0.065 0.087' rpy='0 0 0'/>
+        <origin xyz='-0.007 0.065 -0.087' rpy='0 0 0'/>
         <axis xyz='0 1 0'/>
     </joint>
@@ -34,5 +34,5 @@
         <parent link='left_kingpin_link'/>
         <child link='front_left_wheel_link'/>
-        <origin xyz='-0.007 -0.065 0.087' rpy='0 0 0'/>
+        <origin xyz='-0.007 -0.065 -0.087' rpy='0 0 0'/>
         <axis xyz='0 1 0'/>
     </joint>
@@ -41,5 +41,5 @@
         <parent link='chassis_link'/>
         <child link='rear_right_wheel_link'/>
-        <origin xyz='-1.249 0.589 -0.077' rpy='0 0 0'/>
+        <origin xyz='-1.249 0.589 0.077' rpy='0 0 0'/>
         <axis xyz='0 1 0'/>
     </joint>
@@ -48,5 +48,5 @@
         <parent link='chassis_link'/>
         <child link='rear_left_wheel_link'/>
-        <origin xyz='-1.249 -0.589 -0.077' rpy='0 0 0'/>
+        <origin xyz='-1.249 -0.589 0.077' rpy='0 0 0'/>
         <axis xyz='0 1 0'/>
     </joint>
@@ -55,5 +55,5 @@
         <parent link='chassis_link'/>
         <child link='base_link'/>
-        <origin xyz='-0.741 -0.002 -1.029' rpy='${-pi/2} 0 0'/>
+        <origin xyz='-0.741 -0.002 1.029' rpy='${-pi/2} 0 0'/>
     </joint>
 </robot>

File: src/moa/moa_description/urdf/moa_links.xacro (robot description, xacro)
@@ -12,5 +12,5 @@
                 <color rgba='0.4 0.4 0.4 1'/>
             </material>
-            <origin  xyz='0.281 0 0.133' rpy='${-pi/2} 0 0'/>
+            <origin  xyz='0.281 0 -0.133' rpy='${pi/2} 0 0'/>
         </visual>
     </link>

Commit message: gazebo simulation update

File: src/moa/moa_description/urdf/moa_joints.xacro (robot description, xacro)
@@ -6,4 +6,5 @@
         <child link='chassis_link'/>
         <origin xyz='-0.281 0 0.133' rpy='0 0 0'/>
+        <dynamics damping="10.0" friction="10.0"/>
     </joint>
     <!--Chassis to kingpin1 joint-->
@@ -13,5 +14,6 @@
         <origin xyz='0.288 0.571 0.167' rpy='0 0 0'/>
         <axis xyz='0 0 1'/>
-        <limit lower='${-steering_in}' upper='${steering_out}' velocity='1' effort='25'/>
+        <limit lower='${-steering_in}' upper='${steering_out}' velocity="0.1" effort="1"/>
+        <dynamics damping="10.0" friction="10.0"/>
     </joint>
       <!--Chassis to kingpin2 joint-->
@@ -21,5 +23,6 @@
         <origin xyz='0.288 -0.571 0.167' rpy='0 0 0'/>
         <axis xyz='0 0 1'/>
-        <limit lower='${-steering_out}' upper='${steering_in}' velocity='1' effort='25'/>
+        <limit lower='${-steering_out}' upper='${steering_in}' velocity="0.1" effort="1"/>
+        <dynamics damping="10.0" friction="10.0"/>
     </joint>
     <!--Kingpin1 to wheel joint-->
@@ -29,4 +32,5 @@
         <origin xyz='-0.007 0.065 -0.087' rpy='0 0 0'/>
         <axis xyz='0 1 0'/>
+        <dynamics damping="10.0" friction="10.0"/>
     </joint>
     <!--Kingpin2 to wheel joint-->
@@ -36,4 +40,5 @@
         <origin xyz='-0.007 -0.065 -0.087' rpy='0 0 0'/>
         <axis xyz='0 1 0'/>
+        <dynamics damping="10.0" friction="10.0"/>
     </joint>
     <!--Chassis to wheel joint-->
@@ -43,4 +48,5 @@
         <origin xyz='-1.249 0.589 0.077' rpy='0 0 0'/>
         <axis xyz='0 1 0'/>
+        <dynamics damping="10.0" friction="10.0"/>
     </joint>
     <!--Chassis to wheel joint-->
@@ -50,4 +56,5 @@
         <origin xyz='-1.249 -0.589 0.077' rpy='0 0 0'/>
         <axis xyz='0 1 0'/>
+        <dynamics damping="10.0" friction="10.0"/>
     </joint>
     <!--world to zed base joint-->

File: src/moa/moa_description/urdf/moa_links.xacro (robot description, xacro)
@@ -6,4 +6,5 @@
     <link name='chassis_link'>
         <visual>
+            <origin  xyz='0.281 0 -0.133' rpy='${pi} 0 0'/>
             <geometry>
                 <mesh filename='package://moa_description/meshes/Chassis.stl'/>
@@ -12,19 +13,31 @@
                 <color rgba='0.4 0.4 0.4 1'/>
             </material>
-            <origin  xyz='0.281 0 -0.133' rpy='${pi/2} 0 0'/>
         </visual>
+        <!-- inertial-->
+        <inertial>
+            <mass value="150.0"/>
+            <!-- assumed a box/cubeoid -->
+            <inertia ixx="625.0" ixy="0.0" ixz="0.0" iyy="625.0" iyz="0.0" izz="625.0"/>
+        </inertial>
+        <!-- collision-->
+        <collision>
+            <geometry>
+                <!-- <box size="5.0 5.0 5.0"/> -->
+                <mesh filename='package://moa_description/meshes/Chassis.stl'/>
+            </geometry>
+        </collision>
     </link>
     <!--Wheel/Tyre link-->
     <xacro:tyre_link name='front_right_wheel_link'>
-        <origin xyz='0 0 0' rpy='${pi/2} 0 0'/>
+        <origin xyz='0 0 0' rpy='${pi} 0 0'/>
     </xacro:tyre_link>
     <xacro:tyre_link name='front_left_wheel_link'>
-        <origin xyz='0 0 0' rpy='${-pi/2} 0 0'/>
+        <origin xyz='0 0 0' rpy='0 0 0'/>
     </xacro:tyre_link>
     <xacro:tyre_link name='rear_right_wheel_link'>
-        <origin xyz='0 0 0' rpy='${pi/2} 0 0'/>
+        <origin xyz='0 0 0' rpy='${pi} 0 0'/>
     </xacro:tyre_link>
     <xacro:tyre_link name='rear_left_wheel_link'>
-        <origin xyz='0 0 0' rpy='${-pi/2} 0 0'/>
+        <origin xyz='0 0 0' rpy='0 0 0'/>
     </xacro:tyre_link>
     <!--kingpin link-->

File: src/moa/moa_description/urdf/moa_macro.xacro (robot description, xacro)
@@ -13,12 +13,14 @@
                 </material>
             </visual>
+            <!-- inertial-->
             <inertial>
-                <!-- <origin xyz="0.0 0.0 0.0" rpy="0.0 0.0 0.0"/> -->
                 <mass value="5.0"/>
-                <inertia ixx="0.0" ixy="0.0" ixz="0.0" iyy="0.0" iyz="0.0" izz="0.0"/>
+                <!-- assumed a box/cubeoid -->
+                <inertia ixx="3.33" ixy="0.0" ixz="0.0" iyy="3.33" iyz="0.0" izz="3.33"/>
             </inertial>
+            <!-- collision-->
             <collision>
-                <xacro:insert_block name='origin'/>
                 <geometry>
+                    <!-- <box size="1.0 1.0 1.0"/> -->
                     <mesh filename='package://moa_description/meshes/wheel.stl'/>
                 </geometry>
@@ -35,4 +37,16 @@
                 </geometry>
             </visual>
+            <!-- inertial-->
+            <inertial>
+                <mass value="0.5"/>
+                <!-- assumed solid cylinder -->
+                <inertia ixx="0.00006210" ixy="0.0" ixz="0.0" iyy="0.00006210" iyz="0.0" izz="0.000002520"/>
+            </inertial>
+            <!--collision-->
+            <collision>
+                <geometry>
+                    <cylinder radius='${kingpin_radius}' length='${kingpin_length}'/>
+                </geometry>
+            </collision>
         </link>
     </xacro:macro>

File: src/moa/moa_description/urdf/zed_descr.urdf.xacro (robot description, xacro)
@@ -22,5 +22,5 @@
   <xacro:arg name="cam_pos_y"     default="0.0" />
   <xacro:arg name="cam_pos_z"     default="0.0" />
-  <xacro:arg name="cam_roll"      default="0.0" />
+  <xacro:arg name="cam_roll"      default="1.570796327" />
   <xacro:arg name="cam_pitch"     default="0.0" />
   <xacro:arg name="cam_yaw"       default="0.0" />
